File: EN001-002_MODULO-PSU.kicad_pcb (KiCad board)
At the start: 2 copper layers, 70 x 50 mm, 91 parts, among them J1 2x5P 2.54mm, J2 Conn_01x02, J3 Barrel_Jack_Switch, J5 1x3P 2mm, J6 Conn_01x04, Q1 AO3401, Q10 AO3401, Q11 KY6802, Q13 MMBT2222A, Q2 AO3401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

Commit message: pcb layout
Parts:
- SYM2: value IT000020 -> IT0000__
- moved FID1 32.4 mm to (127.6, 77.5)
- moved R36 5.18 mm to (153.5, 43.9), turned to -90 degrees
- moved C9 0.99 mm to (189.8, 50.5)
- moved J2 0.79 mm to (182.4, 40.0)
- moved SYM2 0.69 mm to (140.7, 79.6)
- moved FID3 0.57 mm to (187.0, 38.3)
- moved C3 0.40 mm to (179.8, 61.4)
- moved D2 0.34 mm to (178.5, 52.1)
- moved D8 0.26 mm to (175.1, 52.4)
- moved JP1 0.22 mm to (157.4, 49.0)
- moved R35 0.21 mm to (175.1, 47.6)
- moved C1 0.13 mm to (188.5, 60.4)
- moved C2 0.09 mm to (180.4, 81.1)
- moved R32 0.06 mm to (181.9, 47.5)
Connections:
- net /INT0# renamed /INT0#_1
- R36 pad 1: Net-(SW1-A) -> Net-(SW1-C)
- SW1 pad 1: Net-(SW1-A) -> GND
- SW1 pad 3: GND -> Net-(SW1-C)
Routing:
- net GND: track 79.8 -> 103.0 mm, vias 59 -> 51
- net /VIN: track 37.8 -> 25.6 mm
- net /VLOGIC: track 99.9 -> 104.9 mm
- net Net-(SW1-C): track 0.00 -> 4.07 mm
- net Net-(SW1-A): track 3.83 -> 0.00 mm
- net /VPOW_EN: track 18.3 -> 21.7 mm
- net /DRIVE: track 50.8 -> 48.3 mm, vias 3 -> 4
- net /VPOW: track 17.9 -> 19.4 mm
- net /VINS: track 52.0 -> 50.7 mm
- net Net-(D8-K): track 3.65 -> 4.59 mm
- net Net-(D1-K): track 11.4 -> 10.8 mm
- net /V_BATT: vias 1 -> 0

Commit message: kicad 8.0.5
Parts:
- moved FID1 0.51 mm to (127.6, 78.0)
- moved FID2 0.13 mm to (194.1, 85.1)
- moved SW1 0.10 mm to (157.5, 39.2)
Routing:
- net /VOUT: track 17.8 -> 20.3 mm
- net /VINS: track 50.7 -> 48.8 mm
- net /VLOGIC: track 104.9 -> 103.7 mm
- net GND: track 103.0 -> 101.8 mm
- net Net-(U1-DRV): track 16.0 -> 15.3 mm
- net /5V#: track 43.0 -> 42.4 mm
- net /DRIVE: track 48.3 -> 47.8 mm
- net /VPOW: track 19.4 -> 18.8 mm
Other:
- board size 70 x 50 mm -> 70.4 x 50.4 mm
- rule pad_to_mask_clearance: 0 -> 0.1

Commit message: Applied schematic mods
Parts:
- removed C5: 10nF, Capacitor_SMD:C_0805_2012Metric_Pad1.18x1.45mm_HandSolder
- added R37: 100k, Resistor_SMD:R_0805_2012Metric_Pad1.20x1.40mm_HandSolder, F.Cu at (117.2, 67.3)
- R26: value 100R -> 100k
Connections:
- net /INT0#_1 renamed /INT0#
- C6 pad 1: Net-(D7-A) -> Net-(D7-K)
- R21 pad 2: /VLOGIC -> /VINS
- R26 pad 1: /DRIVE# -> Net-(Q1-D)
- R26 pad 2: /N1 -> GND
- R31 pad 2: Net-(D7-A) -> Net-(D7-K)
- R7 pad 2: Net-(D7-K) -> Net-(D7-A)
- SW2 pad 1: GND -> Net-(J6-Pin_2)
- U2 pad 10: Net-(D7-A) -> Net-(D7-K)
- U2 pad 2: /N1 -> /DRIVE#
- U2 pad 5: Net-(R23-Pad2) -> /DRIVE
Routing:
- net /N1: track 15.7 -> 0.00 mm
- net (no net): track 0.00 -> 15.7 mm
